File: microkfd.kicad_sch (KiCad schematic)
At the start: 47 parts, among them J1 USB_B_Micro, J2 AVR-ISP-6, J3 OLED, J4 AudioJack3, Q1 MMBT3904, Q2 MMBT3904, SW1 SW_UP, SW2 SW_DN, SW3 SW_ENT, U1 FT231XS, U2 ATmega328P-A, Y1 16MHz

Commit message: finalized 328p design
Parts:
- removed D3, D4: 6.3V, Diode_SMD:D_SOD-323_HandSoldering, symbol Device:D_Zener_Small
- removed J3: OLED, Connector_PinHeader_2.54mm:PinHeader_1x04_P2.54mm_Vertical_SMD_Pin1Right, symbol Connector:Conn_01x04_Female
- removed R10, R11, R16, R5: 10k, Resistor_SMD:R_0603_1608Metric_Pad0.98x0.95mm_HandSolder, symbol Device:R_Small
- removed SW1: SW_UP, Button_Switch_SMD:Panasonic_EVQPUM_EVQPUD, symbol Switch:SW_Push_45deg
- removed SW2: SW_DN, Button_Switch_SMD:Panasonic_EVQPUM_EVQPUD, symbol Switch:SW_Push_45deg
- removed SW3: SW_ENT, Button_Switch_SMD:Panasonic_EVQPUM_EVQPUD, symbol Switch:SW_Push_45deg
- added D3: D_PWR, LED_SMD:LED_0805_2012Metric_Pad1.15x1.40mm_HandSolder, symbol Device:LED_Small_Filled
- added D4, D5: 6.3V, Diode_SMD:D_SOD-323_HandSoldering, symbol Device:D_TVS
- C1: renamed from C2; footprint Capacitor_SMD:C_0603_1608Metric_Pad1.08x0.95mm_HandSolder -> Capacitor_SMD:C_0805_2012Metric_Pad1.18x1.45mm_HandSolder
- C2: renamed from C4; footprint Capacitor_SMD:C_0603_1608Metric_Pad1.08x0.95mm_HandSolder -> Capacitor_SMD:C_0805_2012Metric_Pad1.18x1.45mm_HandSolder
- C3: renamed from C5; footprint Capacitor_SMD:C_0603_1608Metric_Pad1.08x0.95mm_HandSolder -> Capacitor_SMD:C_0805_2012Metric_Pad1.18x1.45mm_HandSolder
- C4: renamed from C6; footprint Capacitor_SMD:C_0603_1608Metric_Pad1.08x0.95mm_HandSolder -> Capacitor_SMD:C_0805_2012Metric_Pad1.18x1.45mm_HandSolder
- C5: renamed from C7; footprint Capacitor_SMD:C_0603_1608Metric_Pad1.08x0.95mm_HandSolder -> Capacitor_SMD:C_0805_2012Metric_Pad1.18x1.45mm_HandSolder
- C6: renamed from C8; footprint Capacitor_SMD:C_0603_1608Metric_Pad1.08x0.95mm_HandSolder -> Capacitor_SMD:C_0805_2012Metric_Pad1.18x1.45mm_HandSolder
- C7: renamed from C9; value 10pF -> 8pF; footprint Capacitor_SMD:C_0603_1608Metric_Pad1.08x0.95mm_HandSolder -> Capacitor_SMD:C_0805_2012Metric_Pad1.18x1.45mm_HandSolder
- C8: renamed from C10; value 10pF -> 8pF; footprint Capacitor_SMD:C_0603_1608Metric_Pad1.08x0.95mm_HandSolder -> Capacitor_SMD:C_0805_2012Metric_Pad1.18x1.45mm_HandSolder
- D1, D2: footprint LED_SMD:LED_0603_1608Metric_Pad1.05x0.95mm_HandSolder -> LED_SMD:LED_0805_2012Metric_Pad1.15x1.40mm_HandSolder
- J1: footprint Connector_USB:USB_Micro-B_Wuerth_629105150521 -> lcsc-comps:U254-051N-4BH83-F1B
- J2: footprint Connector_PinHeader_2.54mm:PinHeader_2x03_P2.54mm_Vertical_SMD -> Connector_PinHeader_2.54mm:PinHeader_1x06_P2.54mm_Vertical
- R1, R12, R13, R14, R15, R17, R18, R2, R3, R6, R7, R8, R9: footprint Resistor_SMD:R_0603_1608Metric_Pad0.98x0.95mm_HandSolder -> Resistor_SMD:R_0805_2012Metric_Pad1.20x1.40mm_HandSolder
- R4: value 10k -> 1k; footprint Resistor_SMD:R_0603_1608Metric_Pad0.98x0.95mm_HandSolder -> Resistor_SMD:R_0805_2012Metric_Pad1.20x1.40mm_HandSolder
- renumbered TP3 to TP1, TP4 to TP2, TP5 to TP3, TP6 to TP4
Connections:
- net GND: now also D3.1 (K), D4.1 (A1), D5.1 (A1)
- net KFD_DATA: now also TP3.1, D4.2 (A2)
- net KFD_SENSE: now also TP4.1, D5.2 (A2)
- net TWI_D_RX: no longer TP3.1
- net TWI_S_RX: no longer TP4.1
- net A0: no longer names the net of U2.23 (PC0)
- net A1: no longer names the net of U2.24 (PC1)
- net A2: no longer names the net of U2.25 (PC2)
- net SCL: no longer names the net of U2.28 (PC5)
- net SDA: no longer names the net of U2.27 (PC4)
- net SDA: no longer R4.1
- new net: D3.2 (A), R4.1
- no-connect marks 14 -> 19
Other:
- moved on the sheet: C7, C8, R17, R18, Y1
