File: microkfd.kicad_sch (KiCad schematic)
At the start: 40 parts, among them J1 USB_B_Micro, J2 AVR-ISP-6, J4 AudioJack3, Q1 MMBT3904, Q2 MMBT3904, U1 FT231XS, U2 ATmega328P-A, Y1 16MHz

Commit message: final rev F DFM updates
Parts:
- removed J1: USB_B_Micro, lcsc-comps:U254-051N-4BH83-F1B, symbol Connector:USB_B_Micro
- removed J4: AudioJack3, Connector_Audio:Jack_3.5mm_CUI_SJ-3523-SMT_Horizontal, symbol Connector:AudioJack3
- added J1: USB_C_Receptacle_USB2.0, Connector_USB:USB_C_Receptacle_HRO_TYPE-C-31-M-12, symbol Connector:USB_C_Receptacle_USB2.0
- added J3: AudioJack4, lcsc-comps:PJ-616-5A, symbol Connector:AudioJack4
- added R10, R5: 5k1, Resistor_SMD:R_0805_2012Metric_Pad1.20x1.40mm_HandSolder, symbol Device:R_Small
- C1, C3, C4, C5, C6: LCSC (none) -> C28233
- C2: LCSC (none) -> C15850
- C7, C8: value 8pF -> 12pF; LCSC (none) -> C1792
- D1, D2: LCSC (none) -> C84256
- D3: LCSC (none) -> C2297
- D4, D5: LCSC (none) -> C85200
- Q1, Q2: LCSC (none) -> C20526
- R1, R2: LCSC (none) -> C17561
- R12, R13, R4, R6, R7, R8, R9: LCSC (none) -> C17513
- R14, R15, R3: LCSC (none) -> C17414
- R17, R18: LCSC (none) -> C17557
- U1: LCSC (none) -> C132160
- U2: LCSC (none) -> C14877
- Y1: LCSC (none) -> C2149025
Connections:
- net +5V: now also J1.A4 (VBUS), J1.A9 (VBUS), J1.B4 (VBUS), J1.B9 (VBUS)
- net GND: now also J1.A1 (GND), J1.A12 (GND), J1.B1 (GND), J1.B12 (GND), J1.S1 (SHIELD), J3.S, R10.1, R5.1
- net KFD_DATA: now also J3.T
- net KFD_SENSE: now also J3.R1
- net at R2.2: now also J1.A7 (D-), J1.B7 (D-); no longer U1.11 (USBDP)
- net at R1.2: now also J1.A6 (D+), J1.B6 (D+); no longer U1.12 (USBDM)
- net USB_D-: now reaches R2.1
- net USB_D-: now also U1.12 (USBDM)
- net USB_D+: now reaches R1.1
- net USB_D+: now also U1.11 (USBDP)
- new net: J1.A5 (CC1), R5.2
- new net: J1.B5 (CC2), R10.2
- no-connect marks 19 -> 21
Other:
- moved on the sheet: R1, R2

Commit message: updated to revA.1
Parts:
- J1: footprint Connector_USB:USB_C_Receptacle_HRO_TYPE-C-31-M-12 -> lcsc-comps:TYPE-611S-T3; LCSC C165948 -> C2874595
Other:
- title: MicroKFD -> KFDMicro
Changed lines of the file:
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@@
   (paper "USLetter")
   (title_block
-    (title "MicroKFD")
-    (date "2023-01-18")
-    (rev "E")
+    (title "KFDMicro")
+    (date "2023-10-13")
+    (rev "A.1")
     (company "W3AXL")
-    (comment 1 "redesigned to use 328P MCU")
+    (comment 1 "updated to new USB C connector")
   )
   (junction (at 63.5 170.18) (diameter 0) (color 0 0 0 0)
@@
     (property "Reference" "J1" (id 0) (at 45.72 143.51 0))
     (property "Value" "USB_C_Receptacle_USB2.0" (id 1) (at 45.72 146.05 0))
-    (property "Footprint" "Connector_USB:USB_C_Receptacle_HRO_TYPE-C-31-M-12" (id 2) (at 49.53 166.37 0)
+    (property "Footprint" "lcsc-comps:TYPE-611S-T3" (id 2) (at 49.53 166.37 0)
       (effects (font (size 1.27 1.27)) hide)
     )
@@
       (effects (font (size 1.27 1.27)) hide)
     )
-    (property "LCSC" "C165948" (id 4) (at 45.72 166.37 0)
+    (property "LCSC" "C2874595" (id 4) (at 45.72 166.37 0)
       (effects (font (size 1.27 1.27)) hide)
     )
@@
     )
     (path "/fabf7749-ebd0-466d-b1d1-b47115541cf1"
-      (reference "J1") (unit 1) (value "USB_C_Receptacle_USB2.0") (footprint "Connector_USB:USB_C_Receptacle_HRO_TYPE-C-31-M-12")
+      (reference "J1") (unit 1) (value "USB_C_Receptacle_USB2.0") (footprint "lcsc-comps:TYPE-611S-T3")
     )
     (path "/f52ac8d2-9aff-4317-9ba9-5b1cbe8ec425"

Commit message: dfm updates 2024
Parts:
- J1: footprint lcsc-comps:TYPE-611S-T3 -> Connector_USB:USB_C_Receptacle_HRO_TYPE-C-31-M-12
- Y1: footprint Crystal:Crystal_SMD_SeikoEpson_FA238V-4Pin_3.2x2.5mm_HandSoldering -> Crystal:Crystal_SMD_3225-4Pin_3.2x2.5mm

Commit message: rev B hardware updates
Parts:
- removed C4: 0.1uF, Capacitor_SMD:C_0805_2012Metric_Pad1.18x1.45mm_HandSolder, symbol Device:C_Small
- removed R1, R2: 22R, Resistor_SMD:R_0805_2012Metric_Pad1.20x1.40mm_HandSolder, symbol Device:R_Small
- removed R3: 10k, Resistor_SMD:R_0805_2012Metric_Pad1.20x1.40mm_HandSolder, symbol Device:R_Small
- removed U1: FT231XS, Package_SO:SSOP-20_3.9x8.7mm_P0.635mm, symbol Interface_USB:FT231XS
- added C9: 0.1uF, Capacitor_SMD:C_0603_1608Metric, symbol Device:C_Small
- added F1: 200mA, Fuse:Fuse_0603_1608Metric, symbol Device:Polyfuse_Small
- added R11, R16: 10k, Resistor_SMD:R_0603_1608Metric, symbol Device:R_Small
- added U1: USBLC6-2SC6, Package_TO_SOT_SMD:SOT-23-6, symbol Power_Protection:USBLC6-2SC6
- added U3: CP2102N-Axx-xQFN28, Package_DFN_QFN:QFN-28-1EP_5x5mm_P0.5mm_EP3.35x3.35mm, symbol Interface_USB:CP2102N-Axx-xQFN28
- C1, C5, C6, C7, C8: footprint Capacitor_SMD:C_0805_2012Metric_Pad1.18x1.45mm_HandSolder -> Capacitor_SMD:C_0603_1608Metric
- C2: value 10uF -> 1uF; footprint Capacitor_SMD:C_0805_2012Metric_Pad1.18x1.45mm_HandSolder -> Capacitor_SMD:C_0603_1608Metric
- C3: value 0.1uF -> 1uF; footprint Capacitor_SMD:C_0805_2012Metric_Pad1.18x1.45mm_HandSolder -> Capacitor_SMD:C_0603_1608Metric; LCSC C28233 -> C15850
- D1, D2, D3: footprint LED_SMD:LED_0805_2012Metric_Pad1.15x1.40mm_HandSolder -> LED_SMD:LED_0805_2012Metric
- D4, D5: footprint Diode_SMD:D_SOD-323_HandSoldering -> Diode_SMD:D_0603_1608Metric
- J3: footprint lcsc-comps:PJ-616-5A -> Connector_Audio:Jack_3.5mm_KoreanHropartsElec_PJ-320D-4A_Horizontal
- R10, R12, R13, R14, R15, R4, R5, R6, R7, R8, R9: footprint Resistor_SMD:R_0805_2012Metric_Pad1.20x1.40mm_HandSolder -> Resistor_SMD:R_0603_1608Metric
- R17, R18: value 220 -> 150; footprint Resistor_SMD:R_0805_2012Metric_Pad1.20x1.40mm_HandSolder -> Resistor_SMD:R_0603_1608Metric
Connections:
- net +5V: now also F1.2, R11.2, U1.5 (VBUS), U3.7 (VREGIN), U3.8 (VBUS); no longer J1.A4 (VBUS), J1.A9 (VBUS), J1.B4 (VBUS), J1.B9 (VBUS)
- net GND: now also J3.R2, U1.2 (GND), U3.29 (GND), U3.3 (GND)
- net S_RX: now also U3.25 (RXD)
- net S_TX: now also U3.26 (TXD)
- net ~{RESET}: now also C9.2, R11.1
- net at JP1.1 (A): now also U3.28 (~{DTR})
- net at C3.1: now also R16.2, U3.6 (VDD)
- net IN_D-: now reaches J1.A7 (D-), J1.B7 (D-)
- net IN_D-: now also U1.1 (I/O1)
- net at JP1.2 (B): now also C9.1
- net IN_D+: now reaches J1.A6 (D+), J1.B6 (D+)
- net IN_D+: now also U1.3 (I/O2)
- new net: F1.1, J1.A4 (VBUS), J1.A9 (VBUS), J1.B4 (VBUS), J1.B9 (VBUS)
- new net: R16.1, U3.9 (~{RST})
- new net OUT_D+: U1.4 (I/O2), U3.4 (D+)
- new net OUT_D-: U1.6 (I/O1), U3.5 (D-)
- no-connect marks 21 -> 28
Other:
- moved on the sheet: C1, C2, D3, J1, J2, R10, R4, R5
