File: microkfd.kicad_pcb (KiCad board)
At the start: 2 copper layers, 55 x 22.5 mm, 43 parts, among them J1 USB_C_Receptacle_USB2.0, J2 AVR-ISP-6, J3 AudioJack4, Q1 MMBT3904, Q2 MMBT3904, U1 FT231XS, U2 ATmega328P-A, Y1 16MHz

Commit message: updated to revA.1
Parts:
- J1: footprint Connector_USB:USB_C_Receptacle_HRO_TYPE-C-31-M-12 -> lcsc-comps:TYPE-611S-T3
- moved R10 23.5 mm to (113.5, 108.8), turned to 180 degrees
- moved J1 3.95 mm to (99.9, 100.0)
- moved D3 1.25 mm to (97.2, 92.8)
- moved C1 0.75 mm to (108.2, 92.8)
- moved C2 0.75 mm to (103.8, 92.8)
- moved C6 0.75 mm to (106.0, 92.8)
- moved R4 0.75 mm to (101.5, 92.8)
- moved G*** 0.50 mm to (98.2, 108.8)
Routing:
- net Net-(J1-PadB5): track 21.8 -> 18.4 mm, vias 2 -> 0
- net +5V: track 104.6 -> 103.0 mm
- net Net-(D3-Pad2): track 2.26 -> 3.51 mm
- net GND: track 0.22 -> 0.00 mm, vias 59 -> 70
Other:
- board text added: "KFDMicro"
- board text added: "rev A.1 - 41/23"
- board text removed: "MicroKFD"
- board text removed: "rev F - 06/20"

Commit message: dfm updates 2024
Parts:
- J1: footprint lcsc-comps:TYPE-611S-T3 -> Connector_USB:USB_C_Receptacle_HRO_TYPE-C-31-M-12
- Y1: footprint Crystal:Crystal_SMD_SeikoEpson_FA238V-4Pin_3.2x2.5mm_HandSoldering -> Crystal:Crystal_SMD_3225-4Pin_3.2x2.5mm
- moved J1 4.24 mm to (95.7, 100.0)
- moved C7 0.61 mm to (121.0, 108.4)
- moved C8 0.60 mm to (116.2, 103.4)
Routing:
- net unconnected-(J3-PadR2)_1: track 9.00 -> 0.00 mm
- net unconnected-(J3-PadR2): track 0.00 -> 9.00 mm
- net +5V: track 103.0 -> 103.8 mm
Other:
- board text added: "rev A.2 - 43/24"
- board text removed: "rev A.1 - 41/23"

Commit message: rev B hardware updates
Parts:
- removed C4: 0.1uF, Capacitor_SMD:C_0805_2012Metric_Pad1.18x1.45mm_HandSolder
- removed R1, R2: 22R, Resistor_SMD:R_0805_2012Metric_Pad1.20x1.40mm_HandSolder
- removed R3: 10k, Resistor_SMD:R_0805_2012Metric_Pad1.20x1.40mm_HandSolder
- added C9: 0.1uF, Capacitor_SMD:C_0603_1608Metric, F.Cu at (109.2, 95.5)
- added F1: 200mA, Fuse:Fuse_0603_1608Metric, F.Cu at (102.8, 97.3)
- added R11: 10k, Resistor_SMD:R_0603_1608Metric, F.Cu at (106.2, 95.5)
- added R16: 10k, Resistor_SMD:R_0603_1608Metric, F.Cu at (109.2, 104.5)
- added U3: CP2102N-Axx-xQFN28, Package_DFN_QFN:QFN-28-1EP_5x5mm_P0.5mm_EP3.35x3.35mm, F.Cu at (111.2, 100.0)
- C1, C5, C6, C7, C8: footprint Capacitor_SMD:C_0805_2012Metric_Pad1.18x1.45mm_HandSolder -> Capacitor_SMD:C_0603_1608Metric
- C2: value 10uF -> 1uF; footprint Capacitor_SMD:C_0805_2012Metric_Pad1.18x1.45mm_HandSolder -> Capacitor_SMD:C_0603_1608Metric
- C3: value 0.1uF -> 1uF; footprint Capacitor_SMD:C_0805_2012Metric_Pad1.18x1.45mm_HandSolder -> Capacitor_SMD:C_0603_1608Metric
- D1, D2, D3: footprint LED_SMD:LED_0805_2012Metric_Pad1.15x1.40mm_HandSolder -> LED_SMD:LED_0805_2012Metric
- D4, D5: footprint Diode_SMD:D_SOD-323_HandSoldering -> Diode_SMD:D_0603_1608Metric
- J3: footprint lcsc-comps:PJ-616-5A -> Connector_Audio:Jack_3.5mm_KoreanHropartsElec_PJ-320D-4A_Horizontal
- R10, R12, R13, R14, R15, R4, R5, R6, R7, R8, R9: footprint Resistor_SMD:R_0805_2012Metric_Pad1.20x1.40mm_HandSolder -> Resistor_SMD:R_0603_1608Metric
- R17, R18: value 220 -> 150; footprint Resistor_SMD:R_0805_2012Metric_Pad1.20x1.40mm_HandSolder -> Resistor_SMD:R_0603_1608Metric
- U1: value FT231XS -> USBLC6-2SC6; footprint Package_SO:SSOP-20_3.9x8.7mm_P0.635mm -> Package_TO_SOT_SMD:SOT-23-6
- moved R10 11.6 mm to (102.8, 104.5)
- moved R5 10.9 mm to (102.8, 95.5)
- moved TP3 8.25 mm to (136.0, 104.8)
- moved J3 6.10 mm to (142.2, 100.0)
- moved U1 5.75 mm to (103.0, 100.0), turned to 0 degrees
- moved TP4 4.55 mm to (140.3, 104.8)
- moved C3 4.54 mm to (106.0, 104.5), turned to 180 degrees
- moved R6 3.58 mm to (118.2, 95.8), turned to -45 degrees
- moved JP1 2.25 mm to (111.2, 91.2), turned to 180 degrees
- moved R4 2.25 mm to (99.2, 92.8)
- moved C1 2.00 mm to (106.2, 92.8)
- moved R7 1.82 mm to (117.0, 97.0), turned to -45 degrees
- moved C6 1.50 mm to (104.5, 92.8)
- moved G*** 1.03 mm to (98.5, 107.8)
- moved C2 1.00 mm to (102.8, 92.8)
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Connections:
- C3 pad 1: Net-(U1-3V3OUT) -> Net-(U3-VDD)
- J1 pad A4: +5V -> Net-(F1-Pad1)
- J1 pad A6: Net-(J1-D+-PadA6) -> /IN_D+
- J1 pad A7: Net-(J1-D--PadA7) -> /IN_D-
- J1 pad A9: +5V -> Net-(F1-Pad1)
- J1 pad B4: +5V -> Net-(F1-Pad1)
- J1 pad B6: Net-(J1-D+-PadA6) -> /IN_D+
- J1 pad B7: Net-(J1-D--PadA7) -> /IN_D-
- J1 pad B9: +5V -> Net-(F1-Pad1)
- J3 pad R2: unconnected-(J3-PadR2)_1 -> GND
- U1 pad 1: Net-(JP1-A) -> /IN_D-
- U1 pad 2: unconnected-(U1-~{RTS}-Pad2) -> GND
- U1 pad 3: Net-(U1-3V3OUT) -> /IN_D+
- U1 pad 4: S_RX -> /OUT_D+
- U1 pad 5: unconnected-(U1-~{RI}-Pad5) -> +5V
- U1 pad 6: GND -> /OUT_D-
Routing:
- net Net-(J1-D+-PadA6): track 18.6 -> 0.00 mm
- net ~{RESET}: track 10.9 -> 25.5 mm
- net Net-(J1-CC2): track 18.7 -> 4.58 mm
- net Net-(F1-Pad1): track 0.00 -> 13.9 mm
- net Net-(U1-3V3OUT): track 12.1 -> 0.00 mm, vias 3 -> 0
- net Net-(J1-CC1): track 16.2 -> 6.21 mm, vias 2 -> 0
- net Net-(J1-D--PadA7): track 9.96 -> 0.00 mm
- net /IN_D-: track 0.00 -> 9.92 mm, vias 0 -> 2
- net /IN_D+: track 0.00 -> 9.77 mm, vias 0 -> 2
- net unconnected-(J3-PadR2): track 9.00 -> 0.00 mm
- net S_TX: track 16.8 -> 8.67 mm
- net +5V: track 103.8 -> 96.5 mm
- net Net-(U3-VDD): track 0.00 -> 6.60 mm, vias 0 -> 2
- net KFD_DATA: track 10.2 -> 16.7 mm
- net KFD_SENSE: track 14.7 -> 8.62 mm
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Other:
- board text added: "5V"
- board text added: "ACT"
- board text added: "GND"
- board text added: "MI"
- board text added: "MO"
- board text added: "PWR"
- board text added: "SCK"
- board text added: "SNS"
- board text added: "rev B - 23/25"
- board text added: "~{RST}"
- board text removed: "rev A.2 - 43/24"
